Commit message: sim draft one wheel

File: src/mz_models/urdf/mzbot1.urdf.xacro (robot description, xacro)
@@ -1,6 +1,15 @@
 <?xml version="1.0"?>
 <robot name="mzbot1" xmlns:xacro="http://ros.org/wiki/xacro">
+    <!-- Include Gazebo Parameters -->
+    <xacro:include filename="$(find mz_models)/urdf/mzbot1_gazebo.xacro" />
     <link name="base_footprint"/>
     <link name="base_link">
+        <inertial>
+            <origin xyz="0 0 0.04" rpy="0.0 0.25 0.3" />
+            <mass value="8.2573504e-01"/>
+            <inertia ixx="2.2124416e-02" ixy="-1.2294101e-04" ixz="3.4938785e-04"
+                     iyy="2.1193702e-02" iyz="-5.0120904e-05"
+                     izz="2.0064271e-02" />
+        </inertial>
         <visual>
             <origin xyz="0.0 0.0 0.0" rpy="0.0 0.0 0.0"/>
@@ -9,4 +18,10 @@
             </geometry>
         </visual>
+        <collision>
+            <origin xyz="0.0 0.0 0.0" rpy="0.0 0.0 0.0"/>
+            <geometry>
+                <mesh filename="package://mz_models/meshes/base_link.STL"/>
+            </geometry>
+        </collision>
     </link>
     <joint name="based_joint" type="fixed">
@@ -17,3 +32,30 @@
         <limit lower="0.0" upper="0.0" effort="0.0" velocity="0.0"/>
     </joint>
+    <link name="wheel_right_link">
+        <inertial>
+          <origin xyz="0 -0.014 0" rpy="0 0 0" />
+          <mass value="0.0530086090966721" />
+          <inertia ixx="1.88176298336665E-05" ixy="-4.8444933029987E-10" ixz="1.88163708851143E-08"
+                   iyy="3.11510738647764E-05" iyz="-6.93560663069607E-11"
+                   izz="1.8801969558182E-05" />
+        </inertial>
+        <visual>
+          <origin xyz="0 0 0" rpy="1.57 0 0" />
+          <geometry>
+            <mesh filename="package://mz_models/meshes/wheel_right_link.STL" />
+          </geometry>
+        </visual>
+        <collision>
+          <origin xyz="0 -0.015 0" rpy="1.57 0 0" />
+          <geometry>
+            <sphere radius="0.033"/>
+          </geometry>
+        </collision>
+      </link>
+      <joint name="wheel_right_joint" type="continuous">
+        <origin xyz="0 -0.0701101849418637 0" rpy="0 0 0" />
+        <parent link="base_link" />
+        <child link="wheel_right_link" />
+        <axis xyz="0 1 0" />
+      </joint>
 </robot>
